Commit message: Update wrist roll follower mesh scaling in URDF, adjust gripper calibration parameters, and add new script for reading motor steps

File: src/so101_follower_description/urdf/so101_follower.urdf.xacro (robot description, xacro)
@@ -280,5 +280,5 @@
       <origin xyz="5.55112e-17 -0.000218214 0.000949706" rpy="-3.14159 -5.55112e-17 -9.17912e-24"/>
       <geometry>
-        <mesh filename="package://so101_follower_description/meshes/wrist_roll_follower_so101_v1.stl"/>
+        <mesh filename="package://so101_follower_description/meshes/wrist_roll_follower_so101_v1.stl" scale="0.001 0.001 0.001"/>
       </geometry>
       <material name="3d_printed"/>
@@ -287,5 +287,5 @@
       <origin xyz="5.55112e-17 -0.000218214 0.000949706" rpy="-3.14159 -5.55112e-17 -9.17912e-24"/>
       <geometry>
-        <mesh filename="package://so101_follower_description/meshes/wrist_roll_follower_so101_v1.stl"/>
+        <mesh filename="package://so101_follower_description/meshes/wrist_roll_follower_so101_v1.stl" scale="0.001 0.001 0.001"/>
       </geometry>
     </collision>
@@ -320,5 +320,5 @@
     <axis xyz="0 0 1"/>
     <!-- calibrated limits: raw(2047,3489) home(2768) = (-1.110,+1.109) rad -->
-    <limit effort="10" velocity="10" lower="-1.110" upper="1.109"/>
+    <limit effort="10" velocity="10" lower="-0.174533" upper="1.74533"/>
   </joint>
   <transmission name="gripper_trans">
